File: neoheart_v2.kicad_sch (KiCad schematic)
At the start: 39 parts, among them J1 Conn_01x03, Q1 A1SHB, U1 ATtiny816-MNR, U2 TPS61240TDRVRQ1

Commit message: unfinished - revision 2.1
Parts:
- added Q2: BSS138, lib:SOT95P237X112-3N, symbol IRLML2502:IRLML2502
- added Q3: A1SHB, lib:SOT95P237X112-3N, symbol IRLML2502:IRLML2502
- added R4, R5: 10K, Resistor_SMD:R_0402_1005Metric_Pad0.72x0.64mm_HandSolder, symbol Device:R_Small
- added R6: 1K, Resistor_SMD:R_0603_1608Metric, symbol Device:R
- added R7: 10K, Resistor_SMD:R_0603_1608Metric, symbol Device:R
Connections:
- net +3V0: now also Q1.2, U1.4 (VCC), Q2.1, Q3.2, R4.1; no longer C3.1, L1.1, U2.4 (EN), U2.6 (VIN)
- net +5V: now also D1.4 (VDD), D10.4 (VDD), D11.4 (VDD), D12.4 (VDD), D13.4 (VDD), D14.4 (VDD), D15.4 (VDD), D16.4 (VDD), D17.4 (VDD), D18.4 (VDD), D19.4 (VDD), D2.4 (VDD), D20.4 (VDD), D21.4 (VDD), D22.4 (VDD), D23.4 (VDD), D24.4 (VDD), D25.4 (VDD), D3.4 (VDD), D4.4 (VDD), D5.4 (VDD), D6.4 (VDD), D7.4 (VDD), D8.4 (VDD), D9.4 (VDD), R5.1; no longer Q1.2, U1.4 (VCC)
- net GND: now also R7.1
- net IO_LEDS: now also Q2.2, R4.2; no longer D1.3 (DIN)
- net ADC_BAT: now reaches U1.1 (PA2)
- net ADC_BAT: now also R6.1, R7.2
- net TX: now reaches U1.20 (PA1)
- net TX: now also TP4.1
- net IO_MOSFET renamed BOOST_MOSFET
- removed net LED5V: D1.4 (VDD), D10.4 (VDD), D11.4 (VDD), D12.4 (VDD), D13.4 (VDD), D14.4 (VDD), D15.4 (VDD), D16.4 (VDD), D17.4 (VDD), D18.4 (VDD), D19.4 (VDD), D2.4 (VDD), D20.4 (VDD), D21.4 (VDD), D22.4 (VDD), D23.4 (VDD), D24.4 (VDD), D25.4 (VDD), D3.4 (VDD), D4.4 (VDD), D5.4 (VDD), D6.4 (VDD), D7.4 (VDD), D8.4 (VDD), D9.4 (VDD), Q1.3
- net PC3 renamed ADC_MOSFET
- net ADC_MOSFET: now also Q3.1; no longer TP4.1
- new net: Q3.3, R6.2
- new net BOOST_3V0: C3.1, L1.1, Q1.3, U2.4 (EN), U2.6 (VIN)
- new net LED_DATA: D1.3 (DIN), Q2.3, R5.2
- no-connect marks 14 -> 12
Other:
- note added: "BATTERY VOLTAGE READER (ADC)"
- note added: "BOOST CONVERTER MOSFET"
- note added: "LEVEL SHIFTER MOSFET"
- note removed: "MOSFET (power saving)"
- moved on the sheet: BT1, Q1
