File: neoheart_v2.kicad_pcb (KiCad board)
At the start: 2 copper layers, 54.2 x 46.5 mm, 40 parts, among them J1 Conn_01x03, Q1 IRLML2502, U2 TPS61240TDRVRQ1

Commit message: uploaded hardware
Parts:
- L1: value 4,7μH -> MLP2012V4R7MT0S1
- Q1: value IRLML2502 -> A1SHB
- SW-ANIM1: value SW_SPST -> TS-1187A-B-A-B
Changed lines of the file:
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@@
 			)
 		)
+		(property ki_fp_filters "Connector*:*_1x??_*")
+		(sheetname "Principale")
+		(sheetfile "neoheart_v2.kicad_sch")
 		(attr through_hole)
 		(fp_line
@@
 			)
 		)
-		(property "Value" "4,7μH"
+		(property "Value" "MLP2012V4R7MT0S1"
 			(at 0 1.55 -90)
 			(layer "F.Fab")
@@
 			)
 		)
-		(property "Value" "SW_SPST"
+		(property "Value" "TS-1187A-B-A-B"
 			(at 0 3.75 0)
 			(layer "F.Fab")
@@
 			)
 		)
+		(sheetname "Principale")
+		(sheetfile "neoheart_v2.kicad_sch")
 		(attr smd)
 		(fp_poly
@@
 			(net 49 "unconnected-(D15-DOUT-Pad1)")
 			(pinfunction "DOUT")
-			(pintype "output")
+			(pintype "output+no_connect")
 		)
 		(pad "2" smd rect
@@
 			)
 		)
-		(property "Value" "IRLML2502"
-			(at 4.5774 2.3544 -90)
+		(property "Value" "A1SHB"
+			(at 2.5 1.91 0)
 			(layer "F.Fab")
 			(effects

Commit message: unfinished - revision 2.1
Parts:
- added Q2: BSS138, lib:SOT95P237X112-3N, F.Cu at (50.3, 41.1)
- added Q3: A1SHB, lib:SOT95P237X112-3N, F.Cu at (42.6, 51.8)
- added R4: 10K, Resistor_SMD:R_0402_1005Metric_Pad0.72x0.64mm_HandSolder, F.Cu at (52.6, 45.0)
- added R5: 10K, Resistor_SMD:R_0402_1005Metric_Pad0.72x0.64mm_HandSolder, F.Cu at (52.6, 47.0)
- added R6: 1K, Resistor_SMD:R_0603_1608Metric, F.Cu at (38.0, 48.6)
- added R7: 10K, Resistor_SMD:R_0603_1608Metric, F.Cu at (38.0, 51.1)
- moved Q1 8.18 mm to (57.6, 49.5)
Connections:
- C3 pad 1: +3V0 -> /BOOST_3V0
- D1 pad 3: /IO_LEDS -> /LED_DATA
- D1 pad 4: /LED5V -> +5V
- D10 pad 4: /LED5V -> +5V
- D11 pad 4: /LED5V -> +5V
- D12 pad 4: /LED5V -> +5V
- D13 pad 4: /LED5V -> +5V
- D14 pad 4: /LED5V -> +5V
- D15 pad 4: /LED5V -> +5V
- D16 pad 4: /LED5V -> +5V
- D17 pad 4: /LED5V -> +5V
- D18 pad 4: /LED5V -> +5V
- D19 pad 4: /LED5V -> +5V
- D2 pad 4: /LED5V -> +5V
- D20 pad 4: /LED5V -> +5V
- D21 pad 4: /LED5V -> +5V
- D22 pad 4: /LED5V -> +5V
- D23 pad 4: /LED5V -> +5V
- D24 pad 4: /LED5V -> +5V
- D25 pad 4: /LED5V -> +5V
- D3 pad 4: /LED5V -> +5V
- D4 pad 4: /LED5V -> +5V
- D5 pad 4: /LED5V -> +5V
- D6 pad 4: /LED5V -> +5V
- D7 pad 4: /LED5V -> +5V
- D8 pad 4: /LED5V -> +5V
- D9 pad 4: /LED5V -> +5V
- L1 pad 1: +3V0 -> /BOOST_3V0
- Q1 pad 1: /IO_MOSFET -> /BOOST_MOSFET
- Q1 pad 2: +5V -> +3V0
- Q1 pad 3: /LED5V -> /BOOST_3V0
- U2 pad 4: +3V0 -> /BOOST_3V0
- U2 pad 6: +3V0 -> /BOOST_3V0
Routing:
- net /LED5V: track 154.5 -> 0.00 mm
- net +5V: track 43.2 -> 167.5 mm, vias 2 -> 0
- net /IO_LEDS: track 19.5 -> 0.00 mm
- net /PC3: track 12.2 -> 0.00 mm
- net /LED_DATA: track 0.00 -> 6.33 mm
- net /IO_MOSFET: track 8.84 -> 6.04 mm, vias 2 -> 1

Commit message: board revision 2.1
Parts:
- removed BATTERY (CR2032): Battery, Battery:BatteryHolder_Keystone_1060_1x2032
- removed MCU: ATtiny816-M, Package_DFN_QFN:VQFN-20-1EP_3x3mm_P0.4mm_EP1.7x1.7mm
- removed PC3: PC3, TestPoint:TestPoint_Pad_D1.0mm
- removed Q3: A1SHB, lib:SOT95P237X112-3N
- removed R6: 1K, Resistor_SMD:R_0603_1608Metric
- removed R7: 10K, Resistor_SMD:R_0603_1608Metric
- added BT1: Battery, Battery:BatteryHolder_Keystone_1060_1x2032, B.Cu at (50.3, 47.2)
- added MCU1: ATtiny816-MNR, Package_DFN_QFN:VQFN-20-1EP_3x3mm_P0.4mm_EP1.7x1.7mm, F.Cu at (50.2, 53.5)
- added TP1: PC3, TestPoint:TestPoint_Pad_D1.0mm, B.Cu at (66.5, 40.6)
- added TP2: PC3, TestPoint:TestPoint_Pad_D1.0mm, B.Cu at (71.4, 40.6)
- added TP4: PC3, TestPoint:TestPoint_Pad_D1.0mm, F.Cu at (50.2, 61.7)
- moved R5 6.36 mm to (54.0, 40.8), turned to 180 degrees
- moved Q1 4.80 mm to (54.6, 45.8), turned to -90 degrees
- moved R4 2.83 mm to (54.0, 42.6), turned to 180 degrees
Connections:
- J1 pad 3: +5V -> +3V0
- R1 pad 1: +5V -> +3V0
Routing:
- net +3V0: track 26.3 -> 50.6 mm
- net /BOOST_3V0: track 0.00 -> 23.6 mm, vias 0 -> 2
- net /LED_DATA: track 6.33 -> 27.7 mm, vias 0 -> 1
- net /IO_LEDS: track 0.00 -> 16.8 mm, vias 0 -> 2
- net /BOOST_MOSFET: track 0.00 -> 13.3 mm, vias 0 -> 2
- net +5V: track 167.5 -> 179.0 mm, vias 0 -> 1
- net GND: track 264.4 -> 255.0 mm
- net /TX: track 0.00 -> 8.04 mm
- net /IO_MOSFET: track 6.04 -> 0.00 mm, vias 1 -> 0
Other:
- board text added: "+3V"
- board text added: "5V"
- board text added: "BAT (CR2032)"
- board text added: "DATA"
- board text added: "DEBUG:"
- board text added: "MCU"
- board text added: "NEOHEART V2.1"
- board text added: "PA1"
- board text removed: "+5V"

Commit message: updated silkscreen text
Other:
- board text added: "LEDS"
- board text added: "TXD"
- board text removed: "DATA"
- board text removed: "PA1"
Changed lines of the file:
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@@
 		)
 	)
-	(gr_text "DATA"
-		(at 68.888032 39.68 0)
+	(gr_text "LEDS"
+		(at 68.761026 39.68 0)
 		(layer "B.SilkS")
 		(effects
@@
 			(justify left bottom mirror)
 		)
-		(render_cache "DATA" 0
-			(polygon
-				(pts
-					(xy 68.8321 39.51) (xy 68.027564 39.51) (xy 67.711758 39.011256) (xy 68.020237 39.011256) (xy 68.239078 39.350265)
-					(xy 68.523865 39.350265) (xy 68.523865 38.66956) (xy 68.239322 38.66956) (xy 68.020237 39.011256)
-					(xy 67.711758 39.011256) (xy 68.027564 38.509581) (xy 68.8321 38.509581)
-				)
-			)
-			(polygon
-				(pts
-					(xy 67.673412 39.510244) (xy 67.358094 39.510244) (xy 67.358094 39.093077) (xy 66.855687 39.093077)
-					(xy 66.855687 39.510244) (xy 66.546231 39.510244) (xy 66.546231 38.674445) (xy 66.86277 38.674445)
-					(xy 66.86277 38.931632) (xy 67.353942 38.931632) (xy 67.353942 38.674445) (xy 66.86277 38.674445)
-					(xy 66.546231 38.674445) (xy 66.546231 38.514466) (xy 67.673412 38.514466)
-				)
-			)
-			(polygon
-				(pts
-					(xy 65.34822 38.6742) (xy 65.706524 38.6742) (xy 65.706524 39.51) (xy 66.014759 39.51) (xy 66.014759 38.6742)
-					(xy 66.377459 38.6742) (xy 66.515456 38.514466) (xy 65.209978 38.514466)
-				)
-			)
-			(polygon
-				(pts
-					(xy 65.179204 39.510244) (xy 64.863886 39.510244) (xy 64.863886 39.093077) (xy 64.361479 39.093077)
-					(xy 64.361479 39.510244) (xy 64.052023 39.510244) (xy 64.052023 38.674445) (xy 64.368562 38.674445)
-					(xy 64.368562 38.931632) (xy 64.859734 38.931632) (xy 64.859734 38.674445) (xy 64.368562 38.674445)
-					(xy 64.052023 38.674445) (xy 64.052023 38.514466) (xy 65.179204 38.514466)
+		(render_cache "LEDS" 0
+			(polygon
+				(pts
+					(xy 67.726657 39.350265) (xy 67.86612 39.51) (xy 68.705094 39.51) (xy 68.705094 38.514466) (xy 68.396859 38.514466)
+					(xy 68.396859 39.350265)
+				)
+			)
+			(polygon
+				(pts
+					(xy 66.68545 39.353684) (xy 66.545987 39.513663) (xy 67.668527 39.513663) (xy 67.668527 38.513244)
+					(xy 66.5433 38.513244) (xy 66.681298 38.672979) (xy 67.358827 38.672979) (xy 67.358827 38.931632)
+					(xy 66.618283 38.931632) (xy 66.618283 39.096496) (xy 67.358827 39.096496) (xy 67.358827 39.353684)
+				)
+			)
+			(polygon
+				(pts
+					(xy 66.484438 39.51) (xy 65.679902 39.51) (xy 65.364096 39.011256) (xy 65.672575 39.011256) (xy 65.891416 39.350265)
+					(xy 66.176203 39.350265) (xy 66.176203 38.66956) (xy 65.891661 38.66956) (xy 65.672575 39.011256)
+					(xy 65.364096 39.011256) (xy 65.679902 38.509581) (xy 66.484438 38.509581)
+				)
+			)
+			(polygon
+				(pts
+					(xy 64.192952 39.35344) (xy 64.324354 39.50658) (xy 65.215352 39.50658) (xy 65.354571 39.346845)
+					(xy 64.552965 39.346845) (xy 64.505338 39.291646) (xy 64.505338 39.087948) (xy 65.307676 39.087948)
+					(xy 65.307676 38.674933) (xy 65.170411 38.514466) (xy 64.150209 38.514466) (xy 64.286741 38.674445)
+					(xy 64.940823 38.674445) (xy 64.999441 38.740879) (xy 64.999441 38.931632) (xy 64.192952 38.931632)
 				)
 			)
@@
 		)
 	)
-	(gr_text "PA1"
-		(at 48.42 64.01 0)
+	(gr_text "TXD"
+		(at 48.324013 64.01 0)
 		(layer "F.SilkS")
 		(effects
@@
 			(justify left bottom)
 		)
-		(render_cache "PA1" 0
-			(polygon
-				(pts
-					(xy 49.576489 63.499769) (xy 48.785631 63.499769) (xy 48.785631 63.847083) (xy 48.475931 63.847083)
-					(xy 48.475931 63.011039) (xy 48.7827 63.011039) (xy 48.7827 63.33979) (xy 49.267034 63.33979) (xy 49.267034 63.011039)
-					(xy 48.7827 63.011039) (xy 48.475931 63.011039) (xy 48.475931 62.851304) (xy 49.576489 62.851304)
-				)
-			)
-			(polygon
-				(pts
-					(xy 50.799902 63.840244) (xy 50.490446 63.840244) (xy 50.490446 63.423077) (xy 49.988039 63.423077)
-					(xy 49.988039 63.840244) (xy 49.672721 63.840244) (xy 49.672721 63.004445) (xy 49.992191 63.004445)
-					(xy 49.992191 63.261632) (xy 50.483363 63.261632) (xy 50.483363 63.004445) (xy 49.992191 63.004445)
-					(xy 49.672721 63.004445) (xy 49.672721 62.844466) (xy 50.799902 62.844466)
-				)
-			)
-			(polygon
-				(pts
-					(xy 51.096168 62.979532) (xy 50.845575 62.839581) (xy 51.402937 62.839581) (xy 51.402937 63.664389)
-					(xy 51.096168 63.960655)
-				)
-			)
+		(render_cache "TXD" 0
+			(polygon
+				(pts
+					(xy 49.481968 63.0042) (xy 49.123664 63.0042) (xy 49.123664 63.84) (xy 48.815429 63.84) (xy 48.815429 63.0042)
+					(xy 48.452728 63.0042) (xy 48.314731 62.844466) (xy 49.620209 62.844466)
+				)
+			)
+			(polygon
+				(pts
+					(xy 50.413999 63.34785) (xy 50.85388 63.84) (xy 50.492645 63.84) (xy 50.234236 63.548618) (xy 49.975827 63.84)
+					(xy 49.617523 63.84) (xy 50.052763 63.34785) (xy 49.610684 62.844466) (xy 49.970209 62.844466)
+					(xy 50.234236 63.14293) (xy 50.496797 62.844466) (xy 50.857788 62.844466)
+				)
+			)
+			(polygon
+				(pts
+					(xy 52.033573 63.341256) (xy 51.717767 63.84) (xy 50.913231 63.84) (xy 50.913231 62.99956) (xy 51.221465 62.99956)
+					(xy 51.221465 63.680265) (xy 51.506253 63.680265) (xy 51.725094 63.341256) (xy 51.506008 62.99956)
+					(xy 51.221465 62.99956) (xy 50.913231 62.99956) (xy 50.913231 62.839581) (xy 51.717767 62.839581)
+				)
+			)

Commit message: revision 2.1, pcbway production files
Routing:
- net GND: track 255.0 -> 261.4 mm
- net /BOOST_MOSFET: track 13.3 -> 16.8 mm
